File: SkyDuino-Hardware.kicad_sch (KiCad schematic)
At the start: 45 parts, among them J1 24V, J2 BT, J4 Drum, J5 Exhaust, J6 Cooling, J7 Cooling, J8 NTC, K1 RT314A24, Q1 DMN6075S, Q2 DMN6075S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

Commit message: Replace L1 with Sunlord SWPA4030S180MT
Parts:
- L1: footprint Inductor_Bourns:L_Bourns_SRN3015BTA -> Inductor_SMD:L_Sunlord_SWPA4030S; LCSC C19947604 -> C96895; LCSC Orig Part C19947604 -> C96895; Manufacturer p/n SRN3015BTA-180M -> SWPA4030S180MT; Mouser https://www.mouser.com/ProductDetail/Bourns/SRN3015BTA-180M -> (none); Mouser p/n 652-SRN3015BTA-180M -> (none)
Changed lines of the file:
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@@
 			)
 		)
-		(property "Footprint" "Inductor_Bourns:L_Bourns_SRN3015BTA"
+		(property "Footprint" "Inductor_SMD:L_Sunlord_SWPA4030S"
 			(at 93.98 30.48 0)
 			(effects
@@
 			)
 		)
-		(property "Datasheet" "https://www.mouser.com/datasheet/2/54/Bourns_08042023_SRN3015BTA_datasheet-3305912.pdf"
+		(property "Datasheet" "https://wmsc.lcsc.com/wmsc/upload/file/pdf/v2/lcsc/2310251551_Sunlord-SWPA4030S180MT_C96895.pdf"
 			(at 93.98 30.48 0)
 			(effects
@@
 			)
 		)
-		(property "Mouser" "https://www.mouser.com/ProductDetail/Bourns/SRN3015BTA-180M"
+		(property "Mouser" ""
 			(at 93.98 30.48 90)
 			(effects
@@
 			)
 		)
-		(property "LCSC" "C19947604"
+		(property "LCSC" "C96895"
 			(at 93.98 30.48 0)
 			(effects
@@
 			)
 		)
-		(property "Mouser p/n" "652-SRN3015BTA-180M"
+		(property "Mouser p/n" ""
 			(at 93.98 30.48 0)
 			(effects
@@
 			)
 		)
-		(property "Manufacturer p/n" "SRN3015BTA-180M"
+		(property "Manufacturer p/n" "SWPA4030S180MT"
 			(at 93.98 30.48 0)
 			(effects
@@
 			)
 		)
-		(property "LCSC Orig Part" "C19947604"
+		(property "LCSC Orig Part" "C96895"
 			(at 93.98 30.48 90)
 			(effects
